Commit message: safety commit

File: models/pole.urdf (robot description, URDF)
Before this commit: robot pole, 1 links, 0 joints
Links:
- link baseLink: geometry collision box size=0.01 0.01 0.5; visual box size=0.01 0.01 0.5

File: models/pole2.urdf (robot description, URDF)
Before this commit: robot pole, 1 links, 0 joints
Links:
- link baseLink: geometry collision box size=0.01 0.01 0.5; visual box size=0.01 0.01 0.5
