Commit message: safety commit

File: models/double_cart_1.urdf (robot description, URDF)
Before this commit: robot cart, 2 links, 1 joints
Links:
- removed link lowerFrictionlessLink
- removed link upperLinkWithFriction
- added link lowerFrictionlessLink1, mass 0.500; collision box size=0.200 0.200 0.025; visual box size=0.200 0.200 0.025
- added link upperLinkWithFriction1, mass 0.500; collision box size=0.200 0.200 0.025; visual box size=0.200 0.200 0.025
Joints:
- removed joint halfBlocksGlue
- added joint halfBlocksGlue1: type fixed, parent upperLinkWithFriction1, child lowerFrictionlessLink1

File: models/double_cart_2.urdf (robot description, URDF)
Before this commit: robot cart, 2 links, 1 joints
Links:
- removed link lowerFrictionlessLink
- removed link upperLinkWithFriction
- added link lowerFrictionlessLink2, mass 0.500; collision box size=0.200 0.200 0.025; visual box size=0.200 0.200 0.025
- added link upperLinkWithFriction2, mass 0.500; collision box size=0.200 0.200 0.025; visual box size=0.200 0.200 0.025
Joints:
- removed joint halfBlocksGlue
- added joint halfBlocksGlue2: type fixed, parent upperLinkWithFriction2, child lowerFrictionlessLink2

File: models/pole1.urdf (robot description, URDF)
Before this commit: robot pole1, 1 links, 0 joints
Links:
- removed link baseLink
- added link baseLinkPole1, mass 5; collision box size=0.010 0.010 0.500; visual box size=0.010 0.010 0.500

File: models/pole2.urdf (robot description, URDF)
Before this commit: robot pole2, 1 links, 0 joints
Links:
- removed link baseLink
- added link baseLinkPole2, mass 5; collision box size=0.010 0.010 0.500; visual box size=0.010 0.010 0.500
