Commit message: safety checkin

File: models/ground.urdf (robot description, URDF)
Before this commit: robot ground, 1 links, 0 joints
Links:
- link baseLink: geometry collision box size=3 3 0.1; visual box size=3 3 0.1

Commit message: safety commit

File: models/ground.urdf (robot description, URDF)
Before this commit: robot ground, 1 links, 0 joints
Links:
- link baseLink: geometry collision box size=3.000 3.000 0.100; visual box size=3.000 3.000 0.100
